File: hardware/droidrefit-pcb/droidrefit-pcb.kicad_sch (KiCad schematic)
At the start: 26 parts, among them J1 USB-C 5V in, J2 SERVO SIG/+5V/GND, J3 NEOPIXEL JST-SH, J5 SPEAKER 4-8ohm, Q1 AO3401A, U1 ESP32-DevKit-30, U2 DFPlayer-Mini, U3 74AHCT1G125

Commit message: PCB: add buttons/buzzer/OLED/UART headers, fix JP1 default pinout
droidrefit-pcb respin closing gaps DESIGN.md had already speced but never
drawn into the schematic/board:

- New J6 (BUTTONS, 1x4: GND/IO32/IO33/IO25), J7 (BUZZER, 1x2: IO27 via a
  new R8 100ohm series/GND), J8 (OLED I2C, 1x4: 3V3/GND/SDA/SCL, with new
  R9/R10 4.7k pull-ups to 3V3), J9 (UART0 ACCESS, 1x4: 3V3/GND/TX0/RX0).
  All four wired straight to U1's existing free socket pins per the pin
  assignments DESIGN.md's own Connectors/firmware-pin-map tables already
  committed to. All dnp+hand-solder like J2/J5 (2.54mm headers, not
  JLC-placed); R8/R9/R10 are real JLC-placed SMD 0603s.
- Fixed JP1 (NeoPixel pin-order solder-bridge field): shipped default was
  DIN-P1/V+-P2/GND-P3, but this session's NeoPixel bring-up empirically
  confirmed the real dome connector is GND-pin1/V+-pin2/Signal-pin3 -- DIN
  and GND were swapped from the shipped default. Remapped which J3 pin each
  bridge pad reaches so the same-row, no-cut default now matches reality.
- Board: placed + routed all new nets (mostly by hand, Freerouting for the
  denser fan-outs), GND pour refilled to pick up the new pads. ERC clean
  (0 errors, same 3 pre-existing symbol-mismatch warnings as before). DRC:
  down to 1 residual error (a zone-clearance short at JP1's own bare/DNP
  bridge-field pads, reproduced across multiple routing strategies -- looks
  like a zone-fill edge case in that one tightly-packed 6-pad SMD cluster,
  not a connectivity mistake; flagged in DESIGN.md/fab/README.md for a
  quick GUI nudge-and-refill before ordering) plus the same 13 pre-existing
  cosmetic warnings as before.
- Deleted the unused, never-instantiated 74xx:74AHCT125 (quad) and
  Connector:Barrel_Jack symbol-library leftovers from the schematic.
- Regenerated the full fab package (gerbers/drill/BOM-full/BOM-JLC/
  CPL-JLC/README) -- BOM-JLC/CPL-JLC now 16 lines/24 designators (was
  11/17). LCSC part numbers for R8/R9/R10 still TBD, not guessed her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
Parts:
- added J6: BUTTONS, Connector_PinHeader_2.54mm:PinHeader_1x04_P2.54mm_Vertical, symbol Connector_Generic:Conn_01x04
- added J7: BUZZER, Connector_PinHeader_2.54mm:PinHeader_1x02_P2.54mm_Vertical, symbol Connector_Generic:Conn_01x02
- added J8: OLED I2C, Connector_PinHeader_2.54mm:PinHeader_1x04_P2.54mm_Vertical, symbol Connector_Generic:Conn_01x04
- added J9: UART0 ACCESS, Connector_PinHeader_2.54mm:PinHeader_1x04_P2.54mm_Vertical, symbol Connector_Generic:Conn_01x04
- added R10, R9: 4.7k, Resistor_SMD:R_0603_1608Metric, symbol Device:R
- added R8: 100, Resistor_SMD:R_0603_1608Metric, symbol Device:R
Connections:
- net GND: now also J6.1 (Pin_1), J7.2 (Pin_2), J8.2 (Pin_2), J9.2 (Pin_2)
- net NPX_P1: now also JP1.6 (P3); no longer JP1.4 (P1)
- net NPX_P3: now also JP1.4 (P1); no longer JP1.6 (P3)
- net BUZZER_IO27: now reaches U1.10 (IO27)
- net BUZZER_IO27: now also R8.1
- net I2C_SCL: now reaches U1.17 (IO22)
- net I2C_SCL: now also J8.4 (Pin_4), R10.1
- net UART0_TX0: now reaches U1.18 (IO1_TX0)
- net UART0_TX0: now also J9.3 (Pin_3)
- net UART0_RX0: now reaches U1.19 (IO3_RX0)
- net UART0_RX0: now also J9.4 (Pin_4)
- net I2C_SDA: now reaches U1.20 (IO21)
- net I2C_SDA: now also J8.3 (Pin_3), R9.1
- net 3V3: now reaches U1.30 (3V3)
- net 3V3: now also J8.1 (Pin_1), J9.1 (Pin_1), R10.2, R9.2
- net BTN_UP: now reaches U1.6 (IO32)
- net BTN_UP: now also J6.2 (Pin_2)
- net BTN_DOWN: now reaches U1.7 (IO33)
- net BTN_DOWN: now also J6.3 (Pin_3)
- net BTN_SND: now reaches U1.8 (IO25)
- net BTN_SND: now also J6.4 (Pin_4)
- new net BUZZER_PWM: J7.1 (Pin_1), R8.2
- no-connect marks 36 -> 31
