File: hardware/droidrefit-pcb/droidrefit-pcb.kicad_sch (KiCad schematic)
At the start: 33 parts, among them J1 USB-C 5V in, J2 SERVO SIG/+5V/GND, J3 NEOPIXEL JST-SH, J5 SPEAKER 4-8ohm, J6 BUTTONS, J7 BUZZER, J8 OLED I2C, J9 UART0 ACCESS, Q1 AO3401A, U1 ESP32-DevKit-30, U2 DFPlayer-Mini, U3 74AHCT1G125

Commit message: PCB: LCSC parts for R8/R9/R10, final fab package regen
- R8 = C22775 (100 ohm 0603 1%, UNI ROYAL 0603WAF1000T5E, JLC Basic)
- R9/R10 = C23162 (4.7k 0603 1%, UNI ROYAL 0603WAF4701T5E, JLC Basic)
  Same UNI ROYAL 0603WAFxxxxT5E family as R1-R7; both Basic, no extended fee.
  Added LCSC/MPN/Manufacturer/JLCPCB_Assembly props to the sch.

- Full fab package regenerated via kicad-cli (GUI-parity engine) from the
  final board: gerbers + zip, drill + maps, 2d-top.png, fab-preview.svg.
  BOM-JLC / CPL-JLC / BOM-full rebuilt to the original hand-crafted JLC
  formats (Designator,Mid X,Mid Y,Layer,Rotation for CPL; comma-separated
  designators for BOM; C1-C4 out of both JLC files; J6-J9 hand-solder).
  Now 14 BOM lines / 20 placed designators (was 11 / 17).

kicad-cli: DRC 0 errors / 0 unconnected, ERC 0 errors. Board is
order-ready.

Co-Authored-By: Claude Sonnet 5 <noreply@anthropic.com>
Parts:
- R10, R9: JLCPCB_Assembly (none) -> Basic; LCSC (none) -> C23162; MPN (none) -> 0603WAF4701T5E; Manufacturer (none) -> UNI ROYAL
- R8: JLCPCB_Assembly (none) -> Basic; LCSC (none) -> C22775; MPN (none) -> 0603WAF1000T5E; Manufacturer (none) -> UNI ROYAL
Changed lines of the file:
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@@
 			)
 		)
+    (property "LCSC" "C23162" (at 139.7 39.37 0)
+      (effects (font (size 1.27 1.27)) (hide yes))
+    )
+    (property "MPN" "0603WAF4701T5E" (at 139.7 39.37 0)
+      (effects (font (size 1.27 1.27)) (hide yes))
+    )
+    (property "Manufacturer" "UNI ROYAL" (at 139.7 39.37 0)
+      (effects (font (size 1.27 1.27)) (hide yes))
+    )
+    (property "JLCPCB_Assembly" "Basic" (at 139.7 39.37 0)
+      (effects (font (size 1.27 1.27)) (hide yes))
+    )
 		(pin "1"
 		)
@@
 			)
 		)
+    (property "LCSC" "C23162" (at 149.86 39.37 0)
+      (effects (font (size 1.27 1.27)) (hide yes))
+    )
+    (property "MPN" "0603WAF4701T5E" (at 149.86 39.37 0)
+      (effects (font (size 1.27 1.27)) (hide yes))
+    )
+    (property "Manufacturer" "UNI ROYAL" (at 149.86 39.37 0)
+      (effects (font (size 1.27 1.27)) (hide yes))
+    )
+    (property "JLCPCB_Assembly" "Basic" (at 149.86 39.37 0)
+      (effects (font (size 1.27 1.27)) (hide yes))
+    )
 		(pin "1"
 		)
@@
 			)
 		)
+    (property "LCSC" "C22775" (at 95.25 44.45 0)
+      (effects (font (size 1.27 1.27)) (hide yes))
+    )
+    (property "MPN" "0603WAF1000T5E" (at 95.25 44.45 0)
+      (effects (font (size 1.27 1.27)) (hide yes))
+    )
+    (property "Manufacturer" "UNI ROYAL" (at 95.25 44.45 0)
+      (effects (font (size 1.27 1.27)) (hide yes))
+    )
+    (property "JLCPCB_Assembly" "Basic" (at 95.25 44.45 0)
+      (effects (font (size 1.27 1.27)) (hide yes))
+    )
 		(pin "1"
 		)

Commit message: PCB: fix J1 USB-C part - order C2894897 (matches the footprint), not C2765186
The KiCad footprint USB_C_Receptacle_HCTL_HC-TYPE-C-16P-01A is drawn
specifically for LCSC C2894897 (HCTL - the KiCad library cites its
datasheet). The BOM was ordering C2765186 (SHOU HAN, a different brand)
whose shield-tab / mounting-post geometry doesn't match -> J1 "doesn't
line up with the holes" in JLC's assembly preview. Swapped J1 to C2894897.

Co-Authored-By: Claude Sonnet 5 <noreply@anthropic.com>
Parts:
- J1: LCSC C2765186 -> C2894897; MPN TYPE-C 16PIN 2MD -> HC-TYPE-C-16P-01A; Manufacturer Korean Hroparts -> HCTL
Changed lines of the file:
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@@
 			)
 		)
-		(property "LCSC" "C2765186"
+		(property "LCSC" "C2894897"
 			(at 39.37 185.42 0)
 			(hide yes)
@@
 			)
 		)
-		(property "MPN" "TYPE-C 16PIN 2MD"
+		(property "MPN" "HC-TYPE-C-16P-01A"
 			(at 39.37 185.42 0)
 			(hide yes)
@@
 			)
 		)
-		(property "Manufacturer" "Korean Hroparts"
+		(property "Manufacturer" "HCTL"
 			(at 39.37 185.42 0)
 			(hide yes)

Commit message: PCB: revert J1 back to C2765186
C2894897 carries a JLC "difficult part" fee (needs an assembly fixture,
flagged high difficulty). The J1 misalignment in JLC's preview is a CPL
rotation-offset issue - part-independent, both LCSC parts show it - so
there's no reason to eat the fee. Fix is the CPL rotation value.

Co-Authored-By: Claude Sonnet 5 <noreply@anthropic.com>
Parts:
- J1: LCSC C2894897 -> C2765186; MPN HC-TYPE-C-16P-01A -> TYPE-C-16PIN-2MD(073); Manufacturer HCTL -> SHOU HAN
Changed lines of the file:
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@@
 			)
 		)
-		(property "LCSC" "C2894897"
+		(property "LCSC" "C2765186"
 			(at 39.37 185.42 0)
 			(hide yes)
@@
 			)
 		)
-		(property "MPN" "HC-TYPE-C-16P-01A"
+		(property "MPN" "TYPE-C-16PIN-2MD(073)"
 			(at 39.37 185.42 0)
 			(hide yes)
@@
 			)
 		)
-		(property "Manufacturer" "HCTL"
+		(property "Manufacturer" "SHOU HAN"
 			(at 39.37 185.42 0)
 			(hide yes)
